Commit message: ajuste posição camera e garra

File: urdf/mybot.urdf.xacro (robot description, xacro)
@@ -142,5 +142,5 @@
 <!-- camera turtlebot3 insper-->
   <joint name="camera_joint" type="fixed">
-    <origin xyz="0.035 -0.011 0.130" rpy="0 0.0 0"/>
+    <origin xyz="0.05 -0.011 0.138" rpy="0 0.0 0"/>
     <parent link="base_link"/>
     <child link="camera_link"/>
@@ -204,5 +204,5 @@
     <parent link="base_footprint"/>
     <child link="base_link_garra"/>
-    <origin xyz="0.045 0.0 0.115" rpy="0 0 -1.57"/>
+    <origin xyz="0.044 0.005 0.115" rpy="0 0 -1.57"/>
   </joint>
   <link name="base_link_garra">
@@ -215,5 +215,5 @@
       <origin rpy="0 0 0" xyz="0 0 0"/>
       <geometry>
-        <mesh filename="package://mybot_description/meshes/garra/base_link_garra_garra.stl" scale="0.001 0.001 0.001"/>
+        <mesh filename="package://mybot_description/meshes/garra/base_link_garra.stl" scale="0.001 0.001 0.001"/>
       </geometry>
       <material name="silver"/>
@@ -223,5 +223,5 @@
       <origin rpy="0 0 0" xyz="0 0 0"/>
       <geometry>
-        <mesh filename="package://mybot_description/meshes/garra/base_link_garra_garra.stl" scale="0.001 0.001 0.001"/>
+        <mesh filename="package://mybot_description/meshes/garra/base_link_garra.stl" scale="0.001 0.001 0.001"/>
       </geometry>
     </collision>

Commit message: atualização urfd garra

File: urdf/mybot.urdf.xacro (robot description, xacro)
@@ -336,6 +336,6 @@
       <origin rpy="0 0 0" xyz="-0.0037506353032803787 0.05642585700103959 0.0018237999124817317"/>
       <mass value="2.8498940e-03" />
-      <inertia ixx="1.1175580e-05" ixy="-4.2369783e-11" ixz="-5.9381719e-09"
-               iyy="1.1192413e-05" iyz="-1.4400107e-11"
+      <inertia ixx="1.1175580e-05" ixy="0.0" ixz="0.0"
+               iyy="1.1192413e-05" iyz="0.0"
                izz="2.0712558e-05" />
     </inertial>
@@ -359,6 +359,6 @@
       <origin rpy="0 0 0" xyz="0.010935004857829403 0.022288541926215877 0.00183118936157051"/>
       <mass value="0.80e-02" />
-      <inertia ixx="1.1175580e-05" ixy="-4.2369783e-11" ixz="-5.9381719e-09"
-               iyy="1.1192413e-05" iyz="-1.4400107e-11"
+      <inertia ixx="1.1175580e-05" ixy="0.0" ixz="0.0"
+               iyy="1.1192413e-05" iyz="0.0"
                izz="2.0712558e-05" />
     </inertial>
@@ -382,6 +382,6 @@
       <origin rpy="0 0 0" xyz="-0.009562998839609715 0.0191706945123718 0.0023786783548043755"/>
       <mass value="0.80e-03" />
-      <inertia ixx="1.1175580e-05" ixy="-4.2369783e-11" ixz="-5.9381719e-09"
-               iyy="1.1192413e-05" iyz="-1.4400107e-11"
+      <inertia ixx="1.1175580e-05" ixy="0.0" ixz="0.0"
+               iyy="1.1192413e-05" iyz="0.0"
                izz="2.0712558e-05" />
     </inertial>

Commit message: fix pid and colors

File: urdf/mybot.urdf.xacro (robot description, xacro)
@@ -215,13 +215,14 @@
       <origin rpy="0 0 0" xyz="0 0 0"/>
       <geometry>
-        <mesh filename="package://mybot_description/meshes/garra/base_link_garra.stl" scale="0.001 0.001 0.001"/>
-      </geometry>
-      <material name="silver"/>
-      <material/>
+        <mesh filename="package://mybot_description/meshes/garra/base_link_garra.dae" scale="0.001 0.001 0.001"/>
+      </geometry>
+      <gazebo reference="base_link_garra">
+      <material>Gazebo/Black</material>
+    </gazebo>
     </visual>
     <collision>
       <origin rpy="0 0 0" xyz="0 0 0"/>
       <geometry>
-        <mesh filename="package://mybot_description/meshes/garra/base_link_garra.stl" scale="0.001 0.001 0.001"/>
+        <mesh filename="package://mybot_description/meshes/garra/base_link_garra.dae" scale="0.001 0.001 0.001"/>
       </geometry>
     </collision>
@@ -236,13 +237,14 @@
       <origin rpy="0 0 0" xyz="-0.007563 0.0205 -0.001"/>
       <geometry>
-        <mesh filename="package://mybot_description/meshes/garra/lat31.stl" scale="0.001 0.001 0.001"/>
-      </geometry>
-      <material name="silver"/>
-      <material/>
+        <mesh filename="package://mybot_description/meshes/garra/lat31.dae" scale="0.001 0.001 0.001"/>
+      </geometry>
+      <gazebo reference="lat31">
+      <material>Gazebo/Black</material>
+    </gazebo>
     </visual>
     <collision>
       <origin rpy="0 0 0" xyz="-0.007563 0.0205 -0.001"/>
       <geometry>
-        <mesh filename="package://mybot_description/meshes/garra/lat31.stl" scale="0.001 0.001 0.001"/>
+        <mesh filename="package://mybot_description/meshes/garra/lat31.dae" scale="0.001 0.001 0.001"/>
       </geometry>
     </collision>
@@ -257,13 +259,14 @@
       <origin rpy="0 0 0" xyz="0.016 0.0 -0.001"/>
       <geometry>
-        <mesh filename="package://mybot_description/meshes/garra/lat11.stl" scale="0.001 0.001 0.001"/>
-      </geometry>
-      <material name="silver"/>
-      <material/>
+        <mesh filename="package://mybot_description/meshes/garra/lat11.dae" scale="0.001 0.001 0.001"/>
+      </geometry>
+      <gazebo reference="lat11">
+      <material>Gazebo/Black</material>
+    </gazebo>
     </visual>
     <collision>
       <origin rpy="0 0 0" xyz="0.016 0.0 -0.001"/>
       <geometry>
-        <mesh filename="package://mybot_description/meshes/garra/lat11.stl" scale="0.001 0.001 0.001"/>
+        <mesh filename="package://mybot_description/meshes/garra/lat11.dae" scale="0.001 0.001 0.001"/>
       </geometry>
     </collision>
@@ -278,13 +281,14 @@
       <origin rpy="0 0 0" xyz="0.002445 -0.0205 -0.001"/>
       <geometry>
-        <mesh filename="package://mybot_description/meshes/garra/lat21.stl" scale="0.001 0.001 0.001"/>
-      </geometry>
-      <material name="silver"/>
-      <material/>
+        <mesh filename="package://mybot_description/meshes/garra/lat21.dae" scale="0.001 0.001 0.001"/>
+      </geometry>
+      <gazebo reference="lat21">
+      <material>Gazebo/Black</material>
+    </gazebo>
     </visual>
     <collision>
       <origin rpy="0 0 0" xyz="0.002445 -0.0205 -0.001"/>
       <geometry>
-        <mesh filename="package://mybot_description/meshes/garra/lat21.stl" scale="0.001 0.001 0.001"/>
+        <mesh filename="package://mybot_description/meshes/garra/lat21.dae" scale="0.001 0.001 0.001"/>
       </geometry>
     </collision>
@@ -299,13 +303,14 @@
       <origin rpy="0 0 0" xyz="-0.003609 5.8e-05 -0.004"/>
       <geometry>
-        <mesh filename="package://mybot_description/meshes/garra/servo_garra1.stl" scale="0.001 0.001 0.001"/>
-      </geometry>
-      <material name="silver"/>
-      <material/>
+        <mesh filename="package://mybot_description/meshes/garra/servo_garra1.dae" scale="0.001 0.001 0.001"/>
+      </geometry>
+      <gazebo reference="servo_garra1">
+      <material>Gazebo/Black</material>
+    </gazebo>
     </visual>
     <collision>
       <origin rpy="0 0 0" xyz="-0.003609 5.8e-05 -0.004"/>
       <geometry>
-        <mesh filename="package://mybot_description/meshes/garra/servo_garra1.stl" scale="0.001 0.001 0.001"/>
+        <mesh filename="package://mybot_description/meshes/garra/servo_garra1.dae" scale="0.001 0.001 0.001"/>
       </geometry>
     </collision>
@@ -320,13 +325,14 @@
       <origin rpy="0 0 0" xyz="-0.005038 0.0205 -0.0252"/>
       <geometry>
-        <mesh filename="package://mybot_description/meshes/garra/base_camera1.stl" scale="0.001 0.001 0.001"/>
-      </geometry>
-      <material name="silver"/>
-      <material/>
+        <mesh filename="package://mybot_description/meshes/garra/base_camera1.dae" scale="0.001 0.001 0.001"/>
+      </geometry>
+      <gazebo reference="base_camera1">
+      <material>Gazebo/Black</material>
+    </gazebo>
     </visual>
     <collision>
       <origin rpy="0 0 0" xyz="-0.005038 0.0205 -0.0252"/>
       <geometry>
-        <mesh filename="package://mybot_description/meshes/garra/base_camera1.stl" scale="0.001 0.001 0.001"/>
+        <mesh filename="package://mybot_description/meshes/garra/base_camera1.dae" scale="0.001 0.001 0.001"/>
       </geometry>
     </collision>
@@ -343,13 +349,11 @@
       <origin rpy="0 0 0" xyz="-0.027109 -0.009942 -0.014"/>
       <geometry>
-        <mesh filename="package://mybot_description/meshes/garra/garra1garrabraco1.stl" scale="0.001 0.001 0.001"/>
-      </geometry>
-      <material name="silver"/>
-      <material/>
+        <mesh filename="package://mybot_description/meshes/garra/arm.dae" scale="0.001 0.001 0.001"/>
+      </geometry>
     </visual>
     <collision>
       <origin rpy="0 0 0" xyz="-0.027109 -0.009942 -0.014"/>
       <geometry>
-        <mesh filename="package://mybot_description/meshes/garra/garra1garrabraco1.stl" scale="0.001 0.001 0.001"/>
+        <mesh filename="package://mybot_description/meshes/garra/arm.dae" scale="0.001 0.001 0.001"/>
       </geometry>
     </collision>
@@ -366,15 +370,13 @@
       <origin rpy="0 0 0" xyz="-0.023009 -0.086931 -0.0205"/>
       <geometry>
-        <mesh filename="package://mybot_description/meshes/garra/garra1garradireita1.stl" scale="0.001 0.001 0.001"/>
-      </geometry>
-      <material name="silver"/>
-      <material/>
+        <mesh filename="package://mybot_description/meshes/garra/direita.dae" scale="0.001 0.001 0.001"/>
+      </geometry>
     </visual>
     <collision>
       <origin rpy="0 0 0" xyz="-0.023009 -0.086931 -0.0205"/>
       <geometry>
-        <mesh filename="package://mybot_description/meshes/garra/garra1garradireita1.stl" scale="0.001 0.001 0.001"/>
-      </geometry>
-    </collision>
+        <mesh filename="package://mybot_description/meshes/garra/direita.dae" scale="0.001 0.001 0.001"/>
+      </geometry>
+      </collision>
   </link>
   <link name="garra1garraesquerda1">
@@ -389,13 +391,12 @@
       <origin rpy="0 0 0" xyz="-0.006109 -0.088614 -0.0205"/>
       <geometry>
-        <mesh filename="package://mybot_description/meshes/garra/garra1garraesquerda1.stl" scale="0.001 0.001 0.001"/>
-      </geometry>
-      <material name="silver"/>
-      <material/>
+       <mesh filename="package://mybot_description/meshes/garra/esquerda.dae" scale="0.001 0.001 0.001"/>
+      </geometry>
+      <material name="green"/>
     </visual>
     <collision>
       <origin rpy="0 0 0" xyz="-0.006109 -0.088614 -0.0205"/>
       <geometry>
-        <mesh filename="package://mybot_description/meshes/garra/garra1garraesquerda1.stl" scale="0.001 0.001 0.001"/>
+        <mesh filename="package://mybot_description/meshes/garra/esquerda.dae" scale="0.001 0.001 0.001"/>
       </geometry>
     </collision>
