Commit message: bumper

File: urdf/mybot.gazebo.xacro (robot description, xacro)
@@ -124,4 +124,26 @@
     </sensor>
   </gazebo>
+  <!--bumper turtlebot3 insper-->
+  <gazebo reference="bumper_link">
+      <sensor name="contacts" type="contact">
+          <contact>
+            <collision>base_footprint_fixed_joint_lump__base_collision_collision_1</collision>
+          </contact>
+          <plugin name="gazebo_ros_bumper_controller" filename="libgazebo_ros_bumper.so">
+            <always_on>true</always_on>
+            <robotNamespace>/bumper</robotNamespace>
+            <bumperTopicName>bumper_states</bumperTopicName>
+            <frameName>bumper</frameName>
+            <visualize>true</visualize>
+            <update_rate>50.0</update_rate>
+          </plugin>
+      </sensor>
+      <material>Gazebo/Red</material>
+      <mu1>0.1</mu1>
+      <mu2>0.1</mu2>
+      <gravity>true</gravity>
+      <selfCollide>false</selfCollide>
+    </gazebo>
+  <!--camera turtlebot3 insper-->
   <!--link : https://www.raspberrypi.org/documentation/hardware/camera/-->
   <gazebo reference="camera_rgb_frame">

File: urdf/mybot.urdf.xacro (robot description, xacro)
@@ -165,3 +165,31 @@
   </joint>
   <link name="camera_rgb_optical_frame"/>
+<!-- bumper turtlebot3 insper-->
+<link name="bumper_link">
+    <inertial>
+        <origin xyz="0.0 0.0 0.0" rpy="0 1.0 0"/>
+        <mass value="0.0000000001"/>
+        <inertia ixx="0.00000001" ixy="0.00000001" ixz="0.00000001" iyy="0.00000001" iyz="0.00000001" izz="0.00000001"/>
+    </inertial>
+    <visual>
+        <origin xyz="0.0 0.0 0.0" rpy="0.0 1.0 0"/>
+        <geometry>
+            <cylinder radius="0.015" length="0.015"/>
+        </geometry>
+        <material name="red">
+            <color rgba="1.0 0.0 0.0 1.0"/>
+        </material>
+    </visual>
+    <collision name="base_collision">
+        <origin xyz="0.0 0.0 0.0" rpy="0.0 1.0 0.0"/>
+        <geometry>
+            <cylinder radius="0.015" length="0.015"/>
+        </geometry>
+    </collision>
+  </link>
+  <joint name="bumper_joint" type="fixed">
+      <origin xyz="0.05 0.0 0.1" rpy="0.0 0.0 0.0"/>
+      <parent link="base_link"/>
+      <child link="bumper_link"/>
+  </joint>
 </robot>

Commit message: correção possiççao camera e bumper

File: urdf/mybot.gazebo.xacro (robot description, xacro)
@@ -139,5 +139,5 @@
           </plugin>
       </sensor>
-      <material>Gazebo/Red</material>
+      <material>Gazebo/Green</material>
       <mu1>0.1</mu1>
       <mu2>0.1</mu2>

File: urdf/mybot.urdf.xacro (robot description, xacro)
@@ -141,13 +141,19 @@
   </link>
   <joint name="camera_joint" type="fixed">
-    <origin xyz="0.040 -0.011 0.130" rpy="0 0.174 0"/>
+    <origin xyz="0.035 -0.011 0.130" rpy="0 0.0 0"/>
     <parent link="base_link"/>
     <child link="camera_link"/>
   </joint>
   <link name="camera_link">
+    <visual>
+        <origin xyz="0.005 0.011 0.013" rpy="0 0 0"/>
+        <geometry>
+            <box size="0.005 0.030 0.027"/>
+        </geometry>
+    </visual>
     <collision>
       <origin xyz="0.005 0.011 0.013" rpy="0 0 0"/>
       <geometry>
-        <box size="0.015 0.030 0.027"/>
+        <box size="0.005 0.030 0.027"/>
       </geometry>
     </collision>
@@ -189,5 +195,5 @@
   </link>
   <joint name="bumper_joint" type="fixed">
-      <origin xyz="0.05 0.0 0.1" rpy="0.0 0.0 0.0"/>
+      <origin xyz="0.05 0.0 0.01" rpy="0.0 0.0 0.0"/>
       <parent link="base_link"/>
       <child link="bumper_link"/>

Commit message: atualização garra

File: urdf/mybot.gazebo.xacro (robot description, xacro)
@@ -124,26 +124,26 @@
     </sensor>
   </gazebo>
-  <!--bumper turtlebot3 insper-->
+<!--bumper turtlebot3 insper-->
   <gazebo reference="bumper_link">
-      <sensor name="contacts" type="contact">
-          <contact>
-            <collision>base_footprint_fixed_joint_lump__base_collision_collision_1</collision>
-          </contact>
-          <plugin name="gazebo_ros_bumper_controller" filename="libgazebo_ros_bumper.so">
-            <always_on>true</always_on>
-            <robotNamespace>/bumper</robotNamespace>
-            <bumperTopicName>bumper_states</bumperTopicName>
-            <frameName>bumper</frameName>
-            <visualize>true</visualize>
-            <update_rate>50.0</update_rate>
-          </plugin>
-      </sensor>
-      <material>Gazebo/Green</material>
-      <mu1>0.1</mu1>
-      <mu2>0.1</mu2>
-      <gravity>true</gravity>
-      <selfCollide>false</selfCollide>
-    </gazebo>
-  <!--camera turtlebot3 insper-->
+    <sensor name="contacts" type="contact">
+        <contact>
+          <collision>base_footprint_fixed_joint_lump__base_collision_collision_1</collision>
+        </contact>
+        <plugin name="gazebo_ros_bumper_controller" filename="libgazebo_ros_bumper.so">
+          <always_on>true</always_on>
+          <robotNamespace>/bumper</robotNamespace>
+          <bumperTopicName>bumper_states</bumperTopicName>
+          <frameName>bumper</frameName>
+          <visualize>true</visualize>
+          <update_rate>50.0</update_rate>
+        </plugin>
+    </sensor>
+    <material>Gazebo/Green</material>
+    <mu1>0.1</mu1>
+    <mu2>0.1</mu2>
+    <gravity>true</gravity>
+    <selfCollide>false</selfCollide>
+  </gazebo>
+<!--camera turtlebot3 insper-->
   <!--link : https://www.raspberrypi.org/documentation/hardware/camera/-->
   <gazebo reference="camera_rgb_frame">
@@ -179,3 +179,47 @@
     </sensor>
   </gazebo>
+<!--garra turtlebot3 insper-->
+	<!-- ROS Control -->
+	<gazebo>
+		<plugin filename="libgazebo_ros_control.so" name="gazebo_ros_control">
+    <robotNamespace>/mybot</robotNamespace>
+    </plugin>
+	</gazebo>
+	<!-- ROS Transmission -->
+  <transmission name="joint1_tran">
+    <type>transmission_interface/SimpleTransmission</type>
+    <joint name="joint1">
+      <!--<hardwareInterface>PositionJointInterface</hardwareInterface>-->
+      <hardwareInterface>hardware_interface/EffortJointInterface</hardwareInterface>
+    </joint>
+    <actuator name="joint1_actr">
+      <!--<hardwareInterface>PositionJointInterface</hardwareInterface>-->
+      <hardwareInterface>hardware_interface/EffortJointInterface</hardwareInterface>
+      <mechanicalReduction>1</mechanicalReduction>
+    </actuator>
+  </transmission>
+  <transmission name="joint2_tran">
+    <type>transmission_interface/SimpleTransmission</type>
+    <joint name="joint2">
+      <!--<hardwareInterface>PositionJointInterface</hardwareInterface>-->
+      <hardwareInterface>hardware_interface/EffortJointInterface</hardwareInterface>
+    </joint>
+    <actuator name="joint2_actr">
+      <!--<hardwareInterface>PositionJointInterface</hardwareInterface>-->
+      <hardwareInterface>hardware_interface/EffortJointInterface</hardwareInterface>
+      <mechanicalReduction>1</mechanicalReduction>
+    </actuator>
+  </transmission>
+  <transmission name="joint3_tran">
+    <type>transmission_interface/SimpleTransmission</type>
+    <joint name="joint3">
+      <!--<hardwareInterface>PositionJointInterface</hardwareInterface>-->
+      <hardwareInterface>hardware_interface/EffortJointInterface</hardwareInterface>
+    </joint>
+    <actuator name="joint3_actr">
+      <!--<hardwareInterface>PositionJointInterface</hardwareInterface>-->
+      <hardwareInterface>hardware_interface/EffortJointInterface</hardwareInterface>
+      <mechanicalReduction>1</mechanicalReduction>
+    </actuator>
+  </transmission>
 </robot>

File: urdf/mybot.urdf.xacro (robot description, xacro)
@@ -140,4 +140,5 @@
     </inertial>
   </link>
+<!-- camera turtlebot3 insper-->
   <joint name="camera_joint" type="fixed">
     <origin xyz="0.035 -0.011 0.130" rpy="0 0.0 0"/>
@@ -172,5 +173,5 @@
   <link name="camera_rgb_optical_frame"/>
 <!-- bumper turtlebot3 insper-->
-<link name="bumper_link">
+  <link name="bumper_link">
     <inertial>
         <origin xyz="0.0 0.0 0.0" rpy="0 1.0 0"/>
@@ -179,5 +180,5 @@
     </inertial>
     <visual>
-        <origin xyz="0.0 0.0 0.0" rpy="0.0 1.0 0"/>
+        <origin xyz="0.0 0.0 0.0" rpy="0.0 1.57 0"/>
         <geometry>
             <cylinder radius="0.015" length="0.015"/>
@@ -188,5 +189,5 @@
     </visual>
     <collision name="base_collision">
-        <origin xyz="0.0 0.0 0.0" rpy="0.0 1.0 0.0"/>
+        <origin xyz="0.0 0.0 0.0" rpy="0.0 1.57 0.0"/>
         <geometry>
             <cylinder radius="0.015" length="0.015"/>
@@ -195,7 +196,254 @@
   </link>
   <joint name="bumper_joint" type="fixed">
-      <origin xyz="0.05 0.0 0.01" rpy="0.0 0.0 0.0"/>
+      <origin xyz="0.04 0.0 0.015" rpy="0.0 0.0 0.0"/>
       <parent link="base_link"/>
       <child link="bumper_link"/>
   </joint>
+<!-- garra turtlebot3 insper-->
+  <joint name="base_joint_garra" type="fixed">
+    <parent link="base_footprint"/>
+    <child link="base_link_garra"/>
+    <origin xyz="0.045 0.0 0.115" rpy="0 0 -1.57"/>
+  </joint>
+  <link name="base_link_garra">
+    <inertial>
+      <origin rpy="0 0 0" xyz="0.0005 -0.0001 0.002"/>
+      <mass value="0.0001"/>
+      <inertia ixx="1.9768356736455373e-06" ixy="3.3842609487814834e-07" ixz="3.3087224502121107e-23" iyy="2.1568932661454165e-06" iyz="-2.274746684520826e-23" izz="4.120108098287789e-06"/>
+    </inertial>
+    <visual>
+      <origin rpy="0 0 0" xyz="0 0 0"/>
+      <geometry>
+        <mesh filename="package://mybot_description/meshes/garra/base_link_garra_garra.stl" scale="0.001 0.001 0.001"/>
+      </geometry>
+      <material name="silver"/>
+      <material/>
+    </visual>
+    <collision>
+      <origin rpy="0 0 0" xyz="0 0 0"/>
+      <geometry>
+        <mesh filename="package://mybot_description/meshes/garra/base_link_garra_garra.stl" scale="0.001 0.001 0.001"/>
+      </geometry>
+    </collision>
+  </link>
+  <link name="lat31">
+    <inertial>
+      <origin rpy="0 0 0" xyz="-0.005014384312211391 -0.0015000010654330244 0.013948367968184407"/>
+      <mass value="0.0001"/>
+      <inertia ixx="8.662089264671677e-08" ixy="0.0" ixz="1.2947458053521905e-11" iyy="1.3378883884262552e-07" iyz="0.0" izz="4.9622899604909504e-08"/>
+    </inertial>
+    <visual>
+      <origin rpy="0 0 0" xyz="-0.007563 0.0205 -0.001"/>
+      <geometry>
+        <mesh filename="package://mybot_description/meshes/garra/lat31.stl" scale="0.001 0.001 0.001"/>
+      </geometry>
+      <material name="silver"/>
+      <material/>
+    </visual>
+    <collision>
+      <origin rpy="0 0 0" xyz="-0.007563 0.0205 -0.001"/>
+      <geometry>
+        <mesh filename="package://mybot_description/meshes/garra/lat31.stl" scale="0.001 0.001 0.001"/>
+      </geometry>
+    </collision>
+  </link>
+  <link name="lat11">
+    <inertial>
+      <origin rpy="0 0 0" xyz="-0.00149999999999997 0.004954936394439788 0.013948367968184407"/>
+      <mass value="0.0001"/>
+      <inertia ixx="1.3378883884262488e-07" ixy="-2.6469779601696886e-23" ixz="0.0" iyy="8.66208926467172e-08" iyz="1.294745805340279e-11" izz="4.962289960490908e-08"/>
+    </inertial>
+    <visual>
+      <origin rpy="0 0 0" xyz="0.016 0.0 -0.001"/>
+      <geometry>
+        <mesh filename="package://mybot_description/meshes/garra/lat11.stl" scale="0.001 0.001 0.001"/>
+      </geometry>
+      <material name="silver"/>
+      <material/>
+    </visual>
+    <collision>
+      <origin rpy="0 0 0" xyz="0.016 0.0 -0.001"/>
+      <geometry>
+        <mesh filename="package://mybot_description/meshes/garra/lat11.stl" scale="0.001 0.001 0.001"/>
+      </geometry>
+    </collision>
+  </link>
+  <link name="lat21">
+    <inertial>
+      <origin rpy="0 0 0" xyz="0.004954582993387833 0.0014999998509883788 0.013948367968184407"/>
+      <mass value="0.0001"/>
+      <inertia ixx="8.66208926467172e-08" ixy="-3.970466940254533e-23" ixz="1.294745805356161e-11" iyy="1.3378883884262557e-07" iyz="0.0" izz="4.9622899604909715e-08"/>
+    </inertial>
+    <visual>
+      <origin rpy="0 0 0" xyz="0.002445 -0.0205 -0.001"/>
+      <geometry>
+        <mesh filename="package://mybot_description/meshes/garra/lat21.stl" scale="0.001 0.001 0.001"/>
+      </geometry>
+      <material name="silver"/>
+      <material/>
+    </visual>
+    <collision>
+      <origin rpy="0 0 0" xyz="0.002445 -0.0205 -0.001"/>
+      <geometry>
+        <mesh filename="package://mybot_description/meshes/garra/lat21.stl" scale="0.001 0.001 0.001"/>
+      </geometry>
+    </collision>
+  </link>
+  <link name="servo_garra1">
+    <inertial>
+      <origin rpy="0 0 0" xyz="0.0003331581426503209 0.00010673599128592421 0.010000547183940757"/>
+      <mass value="0.001"/>
+      <inertia ixx="6.084896121919108e-06" ixy="7.673237329744245e-10" ixz="2.6844653998574326e-10" iyy="5.525444825215397e-06" iyz="-4.006713086347275e-10" izz="9.353516497648977e-06"/>
+    </inertial>
+    <visual>
+      <origin rpy="0 0 0" xyz="-0.003609 5.8e-05 -0.004"/>
+      <geometry>
+        <mesh filename="package://mybot_description/meshes/garra/servo_garra1.stl" scale="0.001 0.001 0.001"/>
+      </geometry>
+      <material name="silver"/>
+      <material/>
+    </visual>
+    <collision>
+      <origin rpy="0 0 0" xyz="-0.003609 5.8e-05 -0.004"/>
+      <geometry>
+        <mesh filename="package://mybot_description/meshes/garra/servo_garra1.stl" scale="0.001 0.001 0.001"/>
+      </geometry>
+    </collision>
+  </link>
+  <link name="base_camera1">
+    <inertial>
+      <origin rpy="0 0 0" xyz="-0.004389339547781822 0.020361286436828687 0.001500000342726699"/>
+      <mass value="0.0001"/>
+      <inertia ixx="1.9742676232972737e-06" ixy="3.353038926051923e-07" ixz="-1.641126335305207e-21" iyy="2.1544513492515026e-06" iyz="1.1249656330721176e-21" izz="4.115104278945627e-06"/>
+    </inertial>
+    <visual>
+      <origin rpy="0 0 0" xyz="-0.005038 0.0205 -0.0252"/>
+      <geometry>
+        <mesh filename="package://mybot_description/meshes/garra/base_camera1.stl" scale="0.001 0.001 0.001"/>
+      </geometry>
+      <material name="silver"/>
+      <material/>
+    </visual>
+    <collision>
+      <origin rpy="0 0 0" xyz="-0.005038 0.0205 -0.0252"/>
+      <geometry>
+        <mesh filename="package://mybot_description/meshes/garra/base_camera1.stl" scale="0.001 0.001 0.001"/>
+      </geometry>
+    </collision>
+  </link>
+  <link name="garra1garrabraco1">
+    <inertial>
+      <origin rpy="0 0 0" xyz="-0.0037506353032803787 0.05642585700103959 0.0018237999124817317"/>
+      <mass value="2.8498940e-03" />
+      <inertia ixx="1.1175580e-05" ixy="-4.2369783e-11" ixz="-5.9381719e-09"
+               iyy="1.1192413e-05" iyz="-1.4400107e-11"
+               izz="2.0712558e-05" />
+    </inertial>
+    <visual>
+      <origin rpy="0 0 0" xyz="-0.027109 -0.009942 -0.014"/>
+      <geometry>
+        <mesh filename="package://mybot_description/meshes/garra/garra1garrabraco1.stl" scale="0.001 0.001 0.001"/>
+      </geometry>
+      <material name="silver"/>
+      <material/>
+    </visual>
+    <collision>
+      <origin rpy="0 0 0" xyz="-0.027109 -0.009942 -0.014"/>
+      <geometry>
+        <mesh filename="package://mybot_description/meshes/garra/garra1garrabraco1.stl" scale="0.001 0.001 0.001"/>
+      </geometry>
+    </collision>
+  </link>
+  <link name="garra1garradireita1">
+    <inertial>
+      <origin rpy="0 0 0" xyz="0.010935004857829403 0.022288541926215877 0.00183118936157051"/>
+      <mass value="0.80e-02" />
+      <inertia ixx="1.1175580e-05" ixy="-4.2369783e-11" ixz="-5.9381719e-09"
+               iyy="1.1192413e-05" iyz="-1.4400107e-11"
+               izz="2.0712558e-05" />
+    </inertial>
+    <visual>
+      <origin rpy="0 0 0" xyz="-0.023009 -0.086931 -0.0205"/>
+      <geometry>
+        <mesh filename="package://mybot_description/meshes/garra/garra1garradireita1.stl" scale="0.001 0.001 0.001"/>
+      </geometry>
+      <material name="silver"/>
+      <material/>
+    </visual>
+    <collision>
+      <origin rpy="0 0 0" xyz="-0.023009 -0.086931 -0.0205"/>
+      <geometry>
+        <mesh filename="package://mybot_description/meshes/garra/garra1garradireita1.stl" scale="0.001 0.001 0.001"/>
+      </geometry>
+    </collision>
+  </link>
+  <link name="garra1garraesquerda1">
+    <inertial>
+      <origin rpy="0 0 0" xyz="-0.009562998839609715 0.0191706945123718 0.0023786783548043755"/>
+      <mass value="0.80e-03" />
+      <inertia ixx="1.1175580e-05" ixy="-4.2369783e-11" ixz="-5.9381719e-09"
+               iyy="1.1192413e-05" iyz="-1.4400107e-11"
+               izz="2.0712558e-05" />
+    </inertial>
+    <visual>
+      <origin rpy="0 0 0" xyz="-0.006109 -0.088614 -0.0205"/>
+      <geometry>
+        <mesh filename="package://mybot_description/meshes/garra/garra1garraesquerda1.stl" scale="0.001 0.001 0.001"/>
+      </geometry>
+      <material name="silver"/>
+      <material/>
+    </visual>
+    <collision>
+      <origin rpy="0 0 0" xyz="-0.006109 -0.088614 -0.0205"/>
+      <geometry>
+        <mesh filename="package://mybot_description/meshes/garra/garra1garraesquerda1.stl" scale="0.001 0.001 0.001"/>
+      </geometry>
+    </collision>
+  </link>
+  <joint name="Rigid1" type="fixed">
+    <origin rpy="0 0 0" xyz="0.007563 -0.0205 0.001"/>
+    <parent link="base_link_garra"/>
+    <child link="lat31"/>
+  </joint>
+  <joint name="Rigid2" type="fixed">
+    <origin rpy="0 0 0" xyz="-0.016 0.0 0.001"/>
+    <parent link="base_link_garra"/>
+    <child link="lat11"/>
+  </joint>
+  <joint name="Rigid3" type="fixed">
+    <origin rpy="0 0 0" xyz="-0.002445 0.0205 0.001"/>
+    <parent link="base_link_garra"/>
+    <child link="lat21"/>
+  </joint>
+  <joint name="Rigid4" type="fixed">
+    <origin rpy="0 0 0" xyz="0.003609 -5.8e-05 0.004"/>
+    <parent link="base_link_garra"/>
+    <child link="servo_garra1"/>
+  </joint>
+  <joint name="Rigid5" type="fixed">
+    <origin rpy="0 0 0" xyz="-0.002525 0.0 0.0242"/>
+    <parent link="lat31"/>
+    <child link="base_camera1"/>
+  </joint>
+  <joint name="joint1" type="revolute">
+    <origin rpy="0 0 0" xyz="0.0235 0.01 0.01"/>
+    <limit effort="25" lower="-3.14159265359" upper="3.14159265359" velocity="1.5"/>
+    <parent link="servo_garra1"/>
+    <child link="garra1garrabraco1"/>
+    <axis xyz="1.0 0.0 0.0"/>
+  </joint>
+  <joint name="joint2" type="revolute">
+    <origin rpy="0 0 0" xyz="-0.0041 0.076989 0.0065"/>
+    <limit effort="25" lower="-3.14159265359" upper="3.14159265359" velocity="1.5"/>
+    <parent link="garra1garrabraco1"/>
+    <child link="garra1garradireita1"/>
+    <axis xyz="0.0 -0.0 1.0"/>
+  </joint>
+  <joint name="joint3" type="revolute">
+    <origin rpy="0 0 0" xyz="-0.021 0.078672 0.0065"/>
+    <limit effort="25" lower="-3.14159265359" upper="3.14159265359" velocity="1.5"/>
+    <parent link="garra1garrabraco1"/>
+    <child link="garra1garraesquerda1"/>
+    <axis xyz="0.0 -0.0 -1.0"/>
+  </joint>
 </robot>

Commit message: ajuste effort

File: urdf/mybot.gazebo.xacro (robot description, xacro)
@@ -190,9 +190,9 @@
     <type>transmission_interface/SimpleTransmission</type>
     <joint name="joint1">
-      <!--<hardwareInterface>PositionJointInterface</hardwareInterface>-->
+      <!-- <hardwareInterface>hardware_interface/PositionJointInterface</hardwareInterface>-->
       <hardwareInterface>hardware_interface/EffortJointInterface</hardwareInterface>
     </joint>
     <actuator name="joint1_actr">
-      <!--<hardwareInterface>PositionJointInterface</hardwareInterface>-->
+      <!-- <hardwareInterface>hardware_interface/PositionJointInterface</hardwareInterface>-->
       <hardwareInterface>hardware_interface/EffortJointInterface</hardwareInterface>
       <mechanicalReduction>1</mechanicalReduction>
@@ -202,9 +202,9 @@
     <type>transmission_interface/SimpleTransmission</type>
     <joint name="joint2">
-      <!--<hardwareInterface>PositionJointInterface</hardwareInterface>-->
+      <!-- <hardwareInterface>hardware_interface/PositionJointInterface</hardwareInterface>-->
       <hardwareInterface>hardware_interface/EffortJointInterface</hardwareInterface>
     </joint>
     <actuator name="joint2_actr">
-      <!--<hardwareInterface>PositionJointInterface</hardwareInterface>-->
+      <!-- <hardwareInterface>hardware_interface/PositionJointInterface</hardwareInterface>-->
       <hardwareInterface>hardware_interface/EffortJointInterface</hardwareInterface>
       <mechanicalReduction>1</mechanicalReduction>
@@ -214,9 +214,9 @@
     <type>transmission_interface/SimpleTransmission</type>
     <joint name="joint3">
-      <!--<hardwareInterface>PositionJointInterface</hardwareInterface>-->
+      <!-- <hardwareInterface>hardware_interface/PositionJointInterface</hardwareInterface>-->
       <hardwareInterface>hardware_interface/EffortJointInterface</hardwareInterface>
     </joint>
     <actuator name="joint3_actr">
-      <!--<hardwareInterface>PositionJointInterface</hardwareInterface>-->
+      <!-- <hardwareInterface>hardware_interface/PositionJointInterface</hardwareInterface>-->
       <hardwareInterface>hardware_interface/EffortJointInterface</hardwareInterface>
       <mechanicalReduction>1</mechanicalReduction>

File: urdf/mybot.urdf.xacro (robot description, xacro)
@@ -428,5 +428,5 @@
   <joint name="joint1" type="revolute">
     <origin rpy="0 0 0" xyz="0.0235 0.01 0.01"/>
-    <limit effort="25" lower="-3.14159265359" upper="3.14159265359" velocity="1.5"/>
+    <limit effort="1" lower="-1.50" upper="1.5" velocity="0.1"/>
     <parent link="servo_garra1"/>
     <child link="garra1garrabraco1"/>
@@ -435,5 +435,5 @@
   <joint name="joint2" type="revolute">
     <origin rpy="0 0 0" xyz="-0.0041 0.076989 0.0065"/>
-    <limit effort="25" lower="-3.14159265359" upper="3.14159265359" velocity="1.5"/>
+    <limit effort="1" lower="-1" upper="0" velocity="0.1"/>
     <parent link="garra1garrabraco1"/>
     <child link="garra1garradireita1"/>
@@ -442,5 +442,5 @@
   <joint name="joint3" type="revolute">
     <origin rpy="0 0 0" xyz="-0.021 0.078672 0.0065"/>
-    <limit effort="25" lower="-3.14159265359" upper="3.14159265359" velocity="1.5"/>
+    <limit effort="1" lower="-1" upper="0" velocity="0.1"/>
     <parent link="garra1garrabraco1"/>
     <child link="garra1garraesquerda1"/>
