Commit message: garra mimica ok e gazebo e rviz

File: urdf/mybot.gazebo.xacro (robot description, xacro)
@@ -186,4 +186,14 @@
     </plugin>
 	</gazebo>
+  <!-- loading plugin: mimic joints works in gazebo now -->
+  <gazebo>
+    <plugin name="gazebo_gripper_ros_control" filename="libroboticsgroup_gazebo_mimic_joint_plugin.so">
+      <joint>joint2</joint>
+      <mimicJoint>joint3</mimicJoint>
+      <multiplier>1.0</multiplier>
+      <offset>0.0</offset>
+      <hasPID>mybot/gazebo_ros_control/pid_gains/joint3</hasPID>
+    </plugin>
+  </gazebo>
 	<!-- ROS Transmission -->
   <transmission name="joint1_tran">
@@ -215,17 +225,14 @@
     </actuator>
   </transmission>
+  <!--
   <transmission name="joint3_tran">
     <type>transmission_interface/SimpleTransmission</type>
     <joint name="joint3">
-      <!--  <hardwareInterface>hardware_interface/PositionJointInterface</hardwareInterface>-->
       <hardwareInterface>hardware_interface/EffortJointInterface</hardwareInterface>
     </joint>
     <actuator name="joint3_actr">
-      <!--  <hardwareInterface>hardware_interface/PositionJointInterface</hardwareInterface>-->
       <hardwareInterface>hardware_interface/EffortJointInterface</hardwareInterface>
       <mechanicalReduction>1</mechanicalReduction>
-      <!--para teste hardware_interface/PositionJointInterface
-      <motorTorqueConstant>1</motorTorqueConstant>-->
     </actuator>
-  </transmission>
+  </transmission> -->
 </robot>

File: urdf/mybot.urdf.xacro (robot description, xacro)
@@ -440,4 +440,5 @@
     <child link="garra1garradireita1"/>
     <axis xyz="0.0 -0.0 1.0"/>
+    <dynamics damping="0.02" friction="0.0" />
   </joint>
   <joint name="joint3" type="revolute">
@@ -446,5 +447,7 @@
     <parent link="garra1garrabraco1"/>
     <child link="garra1garraesquerda1"/>
+    <mimic joint="joint2" multiplier="1" offset="0" />
     <axis xyz="0.0 -0.0 -1.0"/>
+    <dynamics damping="0.02" friction="0.0" />
   </joint>
 </robot>

Commit message: ajuste PID, ajuste base_link, correção launch joint state

File: urdf/mybot.gazebo.xacro (robot description, xacro)
@@ -132,5 +132,5 @@
         <plugin name="gazebo_ros_bumper_controller" filename="libgazebo_ros_bumper.so">
           <always_on>true</always_on>
-          <robotNamespace>/bumper</robotNamespace>
+        <!--  <robotNamespace>/bumper</robotNamespace> -->
           <bumperTopicName>bumper_states</bumperTopicName>
           <frameName>bumper</frameName>
@@ -183,5 +183,5 @@
 	<gazebo>
 		<plugin filename="libgazebo_ros_control.so" name="gazebo_ros_control">
-    <robotNamespace>/mybot</robotNamespace>
+   <!-- <robotNamespace>/mybot</robotNamespace> -->
     </plugin>
 	</gazebo>
@@ -193,6 +193,26 @@
       <multiplier>1.0</multiplier>
       <offset>0.0</offset>
-      <hasPID>mybot/gazebo_ros_control/pid_gains/joint3</hasPID>
-    </plugin>
+      <!-- <hasPID>mybot/gazebo_ros_control/pid_gains/joint3</hasPID> -->
+      <hasPID>gazebo_ros_control/pid_gains/joint3</hasPID>
+    </plugin>
+  </gazebo>
+<!-- estudar se precisa disso mesmo -->
+  <gazebo reference="garra1garrabraco1">
+    <mu1>0.1</mu1>
+    <mu2>0.1</mu2>
+    <kp>500000.0</kp>
+    <kd>10.0</kd>
+  </gazebo>
+  <gazebo reference="garra1garradireita1">
+    <mu1>0.1</mu1>
+    <mu2>0.1</mu2>
+    <kp>500000.0</kp>
+    <kd>10.0</kd>
+  </gazebo>
+  <gazebo reference="garra1garraesquerda1">
+    <mu1>0.1</mu1>
+    <mu2>0.1</mu2>
+    <kp>500000.0</kp>
+    <kd>10.0</kd>
   </gazebo>
 	<!-- ROS Transmission -->

File: urdf/mybot.urdf.xacro (robot description, xacro)
@@ -202,7 +202,7 @@
 <!-- garra turtlebot3 insper-->
   <joint name="base_joint_garra" type="fixed">
-    <parent link="base_footprint"/>
+    <parent link="base_link"/>
     <child link="base_link_garra"/>
-    <origin xyz="0.044 0.005 0.115" rpy="0 0 -1.57"/>
+    <origin xyz="0.044 0.005 0.108" rpy="0 0 -1.57"/>
   </joint>
   <link name="base_link_garra">

Commit message: ajuste atrito

File: urdf/mybot.gazebo.xacro (robot description, xacro)
@@ -199,20 +199,29 @@
 <!-- estudar se precisa disso mesmo -->
   <gazebo reference="garra1garrabraco1">
-    <mu1>0.1</mu1>
-    <mu2>0.1</mu2>
-    <kp>500000.0</kp>
-    <kd>10.0</kd>
+    <kp>1000000.0</kp>
+    <kd>100.0</kd>
+    <mu1>30.0</mu1>
+    <mu2>30.0</mu2>
+    <maxVel>1.0</maxVel>
+    <minDepth>0.001</minDepth>
+    <material>Gazebo/DarkGrey</material>
   </gazebo>
   <gazebo reference="garra1garradireita1">
-    <mu1>0.1</mu1>
-    <mu2>0.1</mu2>
-    <kp>500000.0</kp>
-    <kd>10.0</kd>
+    <kp>1000000.0</kp>
+    <kd>100.0</kd>
+    <mu1>30.0</mu1>
+    <mu2>30.0</mu2>
+    <maxVel>1.0</maxVel>
+    <minDepth>0.001</minDepth>
+    <material>Gazebo/DarkGrey</material>
   </gazebo>
   <gazebo reference="garra1garraesquerda1">
-    <mu1>0.1</mu1>
-    <mu2>0.1</mu2>
-    <kp>500000.0</kp>
-    <kd>10.0</kd>
+    <kp>1000000.0</kp>
+    <kd>100.0</kd>
+    <mu1>30.0</mu1>
+    <mu2>30.0</mu2>
+    <maxVel>1.0</maxVel>
+    <minDepth>0.001</minDepth>
+    <material>Gazebo/DarkGrey</material>
   </gazebo>
 	<!-- ROS Transmission -->

Commit message: garrinha pintada de verde

File: urdf/mybot.gazebo.xacro (robot description, xacro)
@@ -214,5 +214,5 @@
     <maxVel>1.0</maxVel>
     <minDepth>0.001</minDepth>
-    <material>Gazebo/DarkGrey</material>
+    <material>Gazebo/Green</material>
   </gazebo>
   <gazebo reference="garra1garraesquerda1">
@@ -223,5 +223,5 @@
     <maxVel>1.0</maxVel>
     <minDepth>0.001</minDepth>
-    <material>Gazebo/DarkGrey</material>
+    <material>Gazebo/Green</material>
   </gazebo>
 	<!-- ROS Transmission -->

File: urdf/mybot.urdf.xacro (robot description, xacro)
@@ -184,7 +184,5 @@
             <cylinder radius="0.015" length="0.015"/>
         </geometry>
-        <material name="red">
-            <color rgba="1.0 0.0 0.0 1.0"/>
-        </material>
+      <material name="green"/>
     </visual>
     <collision name="base_collision">
@@ -218,5 +216,4 @@
       </geometry>
       <gazebo reference="base_link_garra">
-      <material>Gazebo/Black</material>
     </gazebo>
     </visual>
@@ -240,5 +237,4 @@
       </geometry>
       <gazebo reference="lat31">
-      <material>Gazebo/Black</material>
     </gazebo>
     </visual>
@@ -262,5 +258,4 @@
       </geometry>
       <gazebo reference="lat11">
-      <material>Gazebo/Black</material>
     </gazebo>
     </visual>
@@ -283,7 +278,4 @@
         <mesh filename="package://mybot_description/meshes/garra/lat21.dae" scale="0.001 0.001 0.001"/>
       </geometry>
-      <gazebo reference="lat21">
-      <material>Gazebo/Black</material>
-    </gazebo>
     </visual>
     <collision>
@@ -305,7 +297,4 @@
         <mesh filename="package://mybot_description/meshes/garra/servo_garra1.dae" scale="0.001 0.001 0.001"/>
       </geometry>
-      <gazebo reference="servo_garra1">
-      <material>Gazebo/Black</material>
-    </gazebo>
     </visual>
     <collision>
@@ -327,7 +316,4 @@
         <mesh filename="package://mybot_description/meshes/garra/base_camera1.dae" scale="0.001 0.001 0.001"/>
       </geometry>
-      <gazebo reference="base_camera1">
-      <material>Gazebo/Black</material>
-    </gazebo>
     </visual>
     <collision>
@@ -372,4 +358,5 @@
         <mesh filename="package://mybot_description/meshes/garra/direita.dae" scale="0.001 0.001 0.001"/>
       </geometry>
+      <material name="green"/>
     </visual>
     <collision>
@@ -390,8 +377,8 @@
     <visual>
       <origin rpy="0 0 0" xyz="-0.006109 -0.088614 -0.0205"/>
+      <material name="green"/>
       <geometry>
        <mesh filename="package://mybot_description/meshes/garra/esquerda.dae" scale="0.001 0.001 0.001"/>
       </geometry>
-      <material name="green"/>
     </visual>
     <collision>
